File: plipbox.kicad_pcb (KiCad board)
At the start: 2 copper layers, 10 parts, among them P1 PWR, P2 PARALLEL_PORT, P3 RS232, U1 MAX3221, U2 ARDUINO_NANO_V3

Commit message: Routed, DRC OK
Routing:
- net /ROUT: track 0.00 -> 31.2 mm
- net /DIN: track 0.00 -> 11.2 mm, vias 0 -> 1
- net GND: track 0.00 -> 8.15 mm, vias 0 -> 4
- net /RIN: track 13.4 -> 14.1 mm
- added copper zone on B.Cu, net GND
Changed lines of the file:
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@@
   (general
     (links 45)
-    (no_connects 42)
+    (no_connects 0)
     (area 0 0 0 0)
     (thickness 1.6)
     (drawings 10)
-    (tracks 138)
+    (tracks 165)
     (zones 0)
     (modules 10)
@@
   (layers
     (0 F.Cu signal)
-    (31 B.Cu signal)
+    (31 B.Cu signal hide)
     (32 B.Adhes user)
     (33 F.Adhes user)
@@
   (segment (start 180.175 115.95) (end 180.175 114.9) (width 0.3) (layer F.Cu) (net 3))
   (segment (start 180.175 114.9) (end 180.575 114.5) (width 0.3) (layer F.Cu) (net 3))
+  (segment (start 176.5 110.05) (end 176.5 108.75) (width 0.3) (layer F.Cu) (net 4))
+  (via (at 176.5 108.75) (size 0.6) (drill 0.4) (layers F.Cu B.Cu) (net 4))
+  (segment (start 180.8 118.25) (end 181.475 117.575) (width 0.3) (layer F.Cu) (net 4))
+  (segment (start 181.475 117.575) (end 181.475 115.95) (width 0.3) (layer F.Cu) (net 4))
+  (segment (start 182.775 110.05) (end 182.775 111.475) (width 0.3) (layer F.Cu) (net 4))
+  (segment (start 182.775 111.475) (end 182.75 111.5) (width 0.3) (layer F.Cu) (net 4))
+  (via (at 182.75 111.5) (size 0.6) (drill 0.4) (layers F.Cu B.Cu) (net 4))
+  (segment (start 180.8 118.25) (end 179.5 118.25) (width 0.3) (layer F.Cu) (net 4))
+  (via (at 179.5 118.25) (size 0.6) (drill 0.4) (layers F.Cu B.Cu) (net 4))
+  (segment (start 176.5 115.95) (end 176.5 116.75) (width 0.3) (layer F.Cu) (net 4))
+  (segment (start 176.5 116.75) (end 176 117.25) (width 0.3) (layer F.Cu) (net 4))
+  (via (at 176 117.25) (size 0.6) (drill 0.4) (layers F.Cu B.Cu) (net 4))
   (segment (start 176.5 114.05) (end 178.525 114.05) (width 0.3) (layer F.Cu) (net 5))
   (segment (start 178.525 114.05) (end 181.475 111.1) (width 0.3) (layer F.Cu) (net 5))
@@
   (segment (start 180.825 115.95) (end 180.825 117) (width 0.3) (layer F.Cu) (net 23))
   (segment (start 180.825 117) (end 180.575 117.25) (width 0.3) (layer F.Cu) (net 23))
-  (segment (start 173 117) (end 175.25 114.75) (width 0.3) (layer F.Cu) (net 24))
-  (segment (start 175.25 114.75) (end 175.25 109) (width 0.3) (layer F.Cu) (net 24))
-  (segment (start 175.25 109) (end 175.75 108.5) (width 0.3) (layer F.Cu) (net 24))
-  (segment (start 175.75 108.5) (end 177.75 108.5) (width 0.3) (layer F.Cu) (net 24))
-  (segment (start 177.75 108.5) (end 178.25 109) (width 0.3) (layer F.Cu) (net 24))
-  (segment (start 178.25 109) (end 178.225 109.025) (width 0.3) (layer F.Cu) (net 24))
-  (segment (start 178.225 109.025) (end 178.225 109.225) (width 0.3) (layer F.Cu) (net 24))
-  (segment (start 178.225 109.225) (end 178.225 110.05) (width 0.3) (layer F.Cu) (net 24))
+  (segment (start 178.225 110.05) (end 178.225 109.025) (width 0.3) (layer F.Cu) (net 24))
+  (segment (start 178.225 109.025) (end 178.25 109) (width 0.3) (layer F.Cu) (net 24))
+  (segment (start 178.25 109) (end 177.25 108) (width 0.3) (layer F.Cu) (net 24))
+  (segment (start 177.25 108) (end 175.75 108) (width 0.3) (layer F.Cu) (net 24))
+  (segment (start 175.75 108) (end 175.25 108.5) (width 0.3) (layer F.Cu) (net 24))
+  (segment (start 175.25 108.5) (end 175.25 114.75) (width 0.3) (layer F.Cu) (net 24))
+  (segment (start 175.25 114.75) (end 173 117) (width 0.3) (layer F.Cu) (net 24))
+  (segment (start 178.225 115.95) (end 178.225 116.475) (width 0.3) (layer F.Cu) (net 25))
+  (segment (start 178.225 116.475) (end 176.45 118.25) (width 0.3) (layer F.Cu) (net 25))
+  (segment (start 171.25 118.5) (end 171.25 121) (width 0.3) (layer F.Cu) (net 25))
+  (segment (start 176.45 118.25) (end 171.5 118.25) (width 0.3) (layer F.Cu) (net 25))
+  (segment (start 171.5 118.25) (end 171.25 118.5) (width 0.3) (layer F.Cu) (net 25))
+  (segment (start 171.25 121) (end 173.25 123) (width 0.3) (layer F.Cu) (net 25))
+  (segment (start 173.25 123) (end 188.25 123) (width 0.3) (layer F.Cu) (net 25))
+  (segment (start 188.25 123) (end 188.76 122.49) (width 0.3) (layer F.Cu) (net 25))
+  (segment (start 188.76 122.49) (end 188.76 121.24) (width 0.3) (layer F.Cu) (net 25))
+  (segment (start 178.225 115.95) (end 178.225 116.525) (width 0.3) (layer F.Cu) (net 25))
+  (segment (start 179.5 114.5) (end 179.5 115.925) (width 0.3) (layer F.Cu) (net 26))
+  (segment (start 179.5 115.925) (end 179.525 115.95) (width 0.3) (layer F.Cu) (net 26))
+  (segment (start 186.22 121.24) (end 186.22 120.84) (width 0.3) (layer B.Cu) (net 26))
+  (segment (start 186.22 120.84) (end 179.88 114.5) (width 0.3) (layer B.Cu) (net 26))
+  (segment (start 179.88 114.5) (end 179.5 114.5) (width 0.3) (layer B.Cu) (net 26))
+  (via (at 179.5 114.5) (size 0.6) (drill 0.4) (layers F.Cu B.Cu) (net 26))
+  (zone (net 4) (net_name GND) (layer B.Cu) (hatch edge 0.508)
+    (connect_pads (clearance 0.508))
+    (min_thickness 0.254)
+    (fill yes (arc_segments 16) (thermal_gap 0.508) (thermal_bridge_width 0.508))
+    (polygon
+      (pts
+        (xy 170 87.5) (xy 225 87.5) (xy 225 124) (xy 170 124)
+      )
+    )
+  )
 )

Commit message: Silkscreen
Other:
- board text added: "1"
- board text added: "5V"
- board text added: "Arduino Nano V3"
- board text added: "DB25M"
- board text added: "GND"
- board text added: "PARALLEL PORT"
- board text added: "RS232"
- board text added: "RX"
- board text added: "TX"
- board text added: "VIN"

Commit message: Fixed DB25M footprint
Parts:
- P2: footprint Keio:DB25M-RA-TH -> kuro:DB25M-RA-TH
Other:
- board text added: "plipbox by lallafa PCB by kuro68k lallafa.de/blog/amiga-projects/plipbox/"

Commit message: Plot
Other:
- board text added: "plipbox by lallafa PCB/RS232 by kuro68k lallafa.de/blog/amiga-projects/plipbox/"
- board text removed: "plipbox by lallafa PCB by kuro68k lallafa.de/blog/amiga-projects/plipbox/"
Changed lines of the file:
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@@
     (links 45)
     (no_connects 0)
-    (area 0 0 0 0)
+    (area 169.899999 80.394999 239.35 131.200001)
     (thickness 1.6)
     (drawings 79)
@@
     (40 Dwgs.User user)
     (41 Cmts.User user)
-    (42 Eco1.User user)
-    (43 Eco2.User user hide)
+    (42 Eco1.User user hide)
+    (43 Eco2.User user)
     (44 Edge.Cuts user)
     (45 Margin user)
@@
     (pad 25 thru_hole circle (at -15.235 -1.42 90) (size 1.7 1.7) (drill 1.1) (layers *.Cu *.Mask))
   )
-  (gr_text "plipbox by lallafa\nPCB by kuro68k\nlallafa.de/blog/amiga-projects/plipbox/" (at 199.75 113) (layer Eco2.User)
+  (gr_text "plipbox by lallafa\nPCB/RS232 by kuro68k\nlallafa.de/blog/amiga-projects/plipbox/" (at 199.75 113) (layer Eco2.User)
     (effects (font (size 1.5 1.5) (thickness 0.3)) (justify mirror))
   )
